Commit message: add init for table top

File: graspqp/assets/allegro/allegro_hand.urdf (robot description, URDF)
Before this commit: robot allegro_hand, 19 links, 18 joints
Joints:
- joint index_joint_0: limit lower=-0.5584889 upper=0.5584889 effort=21. velocity=6.283 -> lower=-0.47 upper=0.47 effort=21. velocity=6.283
- joint index_joint_1: limit lower=-0.2792444 upper=1.727825 effort=21. velocity=6.283 -> lower=-0.196 upper=1.61 effort=21. velocity=6.283
- joint index_joint_2: limit lower=-0.2792444 upper=1.727825 effort=21. velocity=6.283 -> lower=-0.174 upper=1.709 effort=21. velocity=6.283
- joint index_joint_3: limit lower=-0.2792444 upper=1.727825 effort=21. velocity=6.283 -> lower=-0.227 upper=1.618 effort=21. velocity=6.283
- joint middle_joint_0: limit lower=-0.5584889 upper=0.5584889 effort=21. velocity=6.283 -> lower=-0.47 upper=0.47 effort=21. velocity=6.283
- joint middle_joint_1: limit lower=-0.2792444 upper=1.727825 effort=21. velocity=6.283 -> lower=-0.196 upper=1.61 effort=21. velocity=6.283
- joint middle_joint_2: limit lower=-0.2792444 upper=1.727825 effort=21. velocity=6.283 -> lower=-0.174 upper=1.709 effort=21. velocity=6.283
- joint middle_joint_3: limit lower=-0.2792444 upper=1.727825 effort=21. velocity=6.283 -> lower=-0.227 upper=1.618 effort=21. velocity=6.283
- joint ring_joint_0: limit lower=-0.5584889 upper=0.5584889 effort=21. velocity=6.283 -> lower=-0.47 upper=0.47 effort=21. velocity=6.283
- joint ring_joint_1: limit lower=-0.2792444 upper=1.727825 effort=21. velocity=6.283 -> lower=-0.196 upper=1.61 effort=21. velocity=6.283
- joint ring_joint_2: limit lower=-0.2792444 upper=1.727825 effort=21. velocity=6.283 -> lower=-0.174 upper=1.709 effort=21. velocity=6.283
- joint ring_joint_3: limit lower=-0.2792444 upper=1.727825 effort=21. velocity=6.283 -> lower=-0.227 upper=1.618 effort=21. velocity=6.283
- joint thumb_joint_0: limit lower=0.2792444 upper=1.5707499 effort=21. velocity=6.283 -> lower=0.263 upper=1.396 effort=21. velocity=6.283
- joint thumb_joint_1: limit lower=-0.3316028 upper=1.1518834 effort=21. velocity=6.283 -> lower=-0.105 upper=1.163 effort=21. velocity=6.283
- joint thumb_joint_2: limit lower=-0.2792444 upper=1.727825 effort=21. velocity=6.283 -> lower=-0.189 upper=1.644 effort=21. velocity=6.283
- joint thumb_joint_3: limit lower=-0.2792444 upper=1.7627305 effort=21. velocity=6.283 -> lower=-0.162 upper=1.719 effort=21. velocity=6.283
